File: lab4/Lab 1 Exercise 1/Lab 1 Exercise 1.kicad_sch (KiCad schematic)
At the start: 6 parts, among them SW1 SW_SPDT

Commit message: Commiting lab4
Parts:
- C1: footprint (none) -> Capacitor_THT:C_Radial_D5.0mm_H5.0mm_P2.00mm
- D1: footprint (none) -> LED_THT:LED_D5.0mm
- R1, R2: footprint (none) -> Resistor_THT:R_Axial_DIN0516_L15.5mm_D5.0mm_P20.32mm_Horizontal
- SW1: footprint (none) -> Button_Switch_THT:SW_E-Switch_EG1224_SPDT_Angled
- V1: footprint (none) -> Connector_JST:JST_PH_B2B-PH-K_1x02_P2.00mm_Vertical
Changed lines of the file:
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@@
       (effects (font (size 1.27 1.27)) (justify left))
     )
-    (property "Footprint" "" (id 2) (at 155.9052 109.22 0)
+    (property "Footprint" "Capacitor_THT:C_Radial_D5.0mm_H5.0mm_P2.00mm" (id 2) (at 155.9052 109.22 0)
       (effects (font (size 1.27 1.27)) hide)
     )
@@
     (property "Reference" "V1" (id 0) (at 114.935 107.95 0))
     (property "Value" "9 V" (id 1) (at 114.935 110.49 0))
-    (property "Footprint" "" (id 2) (at 114.3 113.03 0)
+    (property "Footprint" "Connector_JST:JST_PH_B2B-PH-K_1x02_P2.00mm_Vertical" (id 2) (at 114.3 113.03 0)
       (effects (font (size 1.27 1.27)) hide)
     )
@@
       (effects (font (size 1.27 1.27)) (justify left))
     )
-    (property "Footprint" "" (id 2) (at 172.212 96.52 90)
+    (property "Footprint" "Resistor_THT:R_Axial_DIN0516_L15.5mm_D5.0mm_P20.32mm_Horizontal" (id 2) (at 172.212 96.52 90)
       (effects (font (size 1.27 1.27)) hide)
     )
@@
       (effects (font (size 1.27 1.27)) (justify right))
     )
-    (property "Footprint" "" (id 2) (at 173.99 111.76 0)
+    (property "Footprint" "LED_THT:LED_D5.0mm" (id 2) (at 173.99 111.76 0)
       (effects (font (size 1.27 1.27)) hide)
     )
@@
     (property "Reference" "SW1" (id 0) (at 142.24 85.09 0))
     (property "Value" "SW_SPDT" (id 1) (at 142.24 87.63 0))
-    (property "Footprint" "" (id 2) (at 142.24 92.71 0)
+    (property "Footprint" "Button_Switch_THT:SW_E-Switch_EG1224_SPDT_Angled" (id 2) (at 142.24 92.71 0)
       (effects (font (size 1.27 1.27)) hide)
     )
@@
     (property "Reference" "R2" (id 0) (at 127 86.36 90))
     (property "Value" "2.2k Ohms" (id 1) (at 127 88.9 90))
-    (property "Footprint" "" (id 2) (at 127 90.932 90)
+    (property "Footprint" "Resistor_THT:R_Axial_DIN0516_L15.5mm_D5.0mm_P20.32mm_Horizontal" (id 2) (at 127 90.932 90)
       (effects (font (size 1.27 1.27)) hide)
     )
@@
   (symbol_instances
     (path "/2613b72d-3be1-43c1-9dc9-cd92caf91b10"
-      (reference "C1") (unit 1) (value "4.7u Ferads") (footprint "")
+      (reference "C1") (unit 1) (value "4.7u Ferads") (footprint "Capacitor_THT:C_Radial_D5.0mm_H5.0mm_P2.00mm")
     )
     (path "/7867f95f-d632-488e-b33e-ffadf7e2c9f1"
-      (reference "D1") (unit 1) (value "LED") (footprint "")
+      (reference "D1") (unit 1) (value "LED") (footprint "LED_THT:LED_D5.0mm")
     )
     (path "/5bbd81b4-ffe7-4871-b4c0-1b1157ecaf80"
-      (reference "R1") (unit 1) (value "20k Ohms") (footprint "")
+      (reference "R1") (unit 1) (value "20k Ohms") (footprint "Resistor_THT:R_Axial_DIN0516_L15.5mm_D5.0mm_P20.32mm_Horizontal")
     )
     (path "/fc75a64c-4936-4d48-b2ed-42ffa2d51c7d"
-      (reference "R2") (unit 1) (value "2.2k Ohms") (footprint "")
+      (reference "R2") (unit 1) (value "2.2k Ohms") (footprint "Resistor_THT:R_Axial_DIN0516_L15.5mm_D5.0mm_P20.32mm_Horizontal")
     )
     (path "/d475b67c-cb0e-4fd5-955a-cbd3bf00eee1"
-      (reference "SW1") (unit 1) (value "SW_SPDT") (footprint "")
+      (reference "SW1") (unit 1) (value "SW_SPDT") (footprint "Button_Switch_THT:SW_E-Switch_EG1224_SPDT_Angled")
     )
     (path "/4649ca04-5806-43bb-acca-d0e920eff663"
-      (reference "V1") (unit 1) (value "9 V") (footprint "")
+      (reference "V1") (unit 1) (value "9 V") (footprint "Connector_JST:JST_PH_B2B-PH-K_1x02_P2.00mm_Vertical")
     )
   )
